Commit message: URDF for smart pneumatic gripper done until gripper base

File: intera_tools_description/urdf/smart_pneumatic_gripper/rethink_pneumatic_gripper.xacro (robot description, xacro)
@@ -8,8 +8,9 @@
 <!-- #ToDo Update distances in meters for pneumatic gripper -->
     <xacro:property name="end_of_arm_offset" value="-0.005" scope="local"/>
-    <xacro:property name="connector_plate_length" value="0.0151" scope="local"/>
+    <xacro:property name="connector_plate_length" value="0.032" scope="local"/>
     <xacro:property name="pneumatic_gripper_base_length" value="0.04552" scope="local"/>
-    <xacro:property name="ft_sensor_lenght" value="0.0001" scope="local"/>
-    <xacro:property name="ft_gripper_adapter_lenght" value="0.0001" scope="local"/>
+    <xacro:property name="ft_sensor_length" value="0.033" scope="local"/>
+    <xacro:property name="adapter_top_length" value="0.013" scope="local"/>
+    <xacro:property name="adapter_bottom_length" value="0.018" scope="local"/>
     <xacro:property name="finger_length" value="0.0021" scope="local"/>
 <!-- Start Kinematic Chain -->
@@ -34,5 +35,5 @@
      <link name="${side}_connector_plate_base">
       <inertial>
-        <origin xyz="0 0 0" rpy="0 0 0" />
+	      <origin xyz="0 0 0" rpy="3.1416 0 0" />
         <mass value="0.0" />
         <inertia ixx="6.9922E-05"  ixy="6.1026E-08"  ixz="-1.7042E-06"
@@ -40,7 +41,7 @@
       </inertial>
       <visual>
-        <origin xyz="0 0 0" rpy="0 0 0" />
-        <geometry>
-		<mesh filename="package://intera_tools_description/meshes/smart_pneumatic_gripper/DAE/ati_9105_t_delta.DAE" />
+        <origin xyz="0 0 0" rpy="3.1416 0 0" />
+        <geometry>
+		<mesh filename="package://intera_tools_description/meshes/smart_pneumatic_gripper/smart_click_adapter.STL" scale="0.001 0.001 0.001" />
         </geometry>
         <material name="black">
@@ -49,7 +50,7 @@
       </visual>
       <collision>
-        <origin xyz="0 0 0.0135" rpy="0 0 0" />
+        <origin xyz="0 0 0.0135" rpy="3.1416 0 0" />
           <geometry>
-            <cylinder length="${connector_plate_length*2.0}" radius="0.04"/>
+            <cylinder length="${connector_plate_length}" radius="0.04"/>
           </geometry>
           <material name="darkred">
@@ -65,9 +66,122 @@
     <!-- Connector Plate base-mount joint -->
     <joint name="${side}_connector_plate_mount_joint" type="fixed">
-      <origin xyz="0 0 0" rpy="0 0 0" />
+	    <origin xyz="0 0 ${connector_plate_length} " rpy="0 0 0" />
       <parent link="${side}_connector_plate_base"  />
       <child  link="${side}_connector_plate_mount" />
     </joint>
+    <!-- Connector Plate mount link -->
     <link name="${side}_connector_plate_mount" />
+    <!-- Connector plate mount-F/T sensor joint -->
+    <joint name="${side}_connector_plate_ft_sensor_joint" type="fixed">
+	    <origin xyz="0 0 0" rpy="0 0 0" />
+      <parent link="${side}_connector_plate_mount"  />
+      <child  link="${side}_ft_sensor_link" />
+    </joint>
+    <!-- F/T sensor link -->
+    <link name="${side}_ft_sensor_link">
+      <visual>
+        <origin xyz="0 0 0" rpy="3.1416 0 0" />
+        <geometry>
+		<mesh filename="package://intera_tools_description/meshes/smart_pneumatic_gripper/ati_9105_t_delta.STL" scale="0.001 0.001 0.001"/>
+        </geometry>
+      </visual>
+      <collision>
+        <origin xyz="0 0 0" rpy="3.1416 0 0" />
+        <geometry>
+		<cylinder length="${ft_sensor_length}" radius="0.046"/>
+        </geometry>
+        <material name="darkred">
+          <color rgba=".5 .1 .1 1"/>
+        </material>
+      </collision>
+      <inertial>
+        <origin rpy="0 0 0" xyz="0.0 0.0 0.0"/>
+        <mass value="2e-06"/>
+        <inertia ixx="1.1e-09" ixy="0" ixz="0" iyy="1.1e-09" iyz="0" izz="1.1e-09"/>
+      </inertial>
+    </link>
+    <!-- F/T Sensor-Adapter Top Part Joint -->
+    <joint name="${side}_ft_sensor_adapter_top_joint" type="fixed">        <origin xyz="0 0 ${ft_sensor_length}" rpy="0 0 0" />                 <parent link="${side}_ft_sensor_link" />
+      <child  link="${side}_adapter_top" />
+    </joint>
+    <!-- Adapter Top Part Link -->
+    <link name="${side}_adapter_top">
+      <visual>
+	      <origin xyz="0 0 ${adapter_top_length}" rpy="${pi/2*-1} 0 0" />
+        <geometry>
+		<mesh filename="package://intera_tools_description/meshes/smart_pneumatic_gripper/ft_gripper_adapter_top.STL" scale="0.001 0.001 0.001"/>
+        </geometry>
+      </visual>
+      <collision>
+	      <origin xyz="0 0 ${adapter_top_length}" rpy="${pi/2*-1} 0 0" />
+        <geometry>
+		<cylinder length="${adapter_top_length}" radius="0.046"/>
+        </geometry>
+        <material name="darkred">
+          <color rgba=".5 .1 .1 1"/>
+        </material>
+      </collision>
+      <inertial>
+        <origin rpy="0 0 0" xyz="0.0 0.0 0.0"/>
+        <mass value="2e-06"/>
+        <inertia ixx="1.1e-09" ixy="0" ixz="0" iyy="1.1e-09" iyz="0" izz="1.1e-09"/>
+      </inertial>
+    </link>
+    <!-- Top-Bottom Adapter Parts Joint -->
+    <joint name="${side}_adapter_top_bottom_joint" type="fixed">        <origin xyz="0 0 ${adapter_top_length}" rpy="0 0 0" />                 <parent link="${side}_adapter_top" />
+      <child  link="${side}_adapter_bottom" />
+    </joint>
+    <!-- Adapter Bottom Part Link -->
+    <link name="${side}_adapter_bottom">
+      <visual>
+	      <origin xyz="0 0 ${adapter_bottom_length}" rpy="${pi/2*-1} 0 0" />
+        <geometry>
+		<mesh filename="package://intera_tools_description/meshes/smart_pneumatic_gripper/ft_gripper_adapter_bottom.STL" scale="0.001 0.001 0.001"/>
+        </geometry>
+      </visual>
+      <collision>
+	      <origin xyz="0 0 ${adapter_bottom_length}" rpy="${pi/2*-1} 0 0" />
+        <geometry>
+		<cylinder length="${adapter_bottom_length}" radius="0.046"/>
+        </geometry>
+        <material name="darkred">
+          <color rgba=".5 .1 .1 1"/>
+        </material>
+      </collision>
+      <inertial>
+        <origin rpy="0 0 0" xyz="0.0 0.0 0.0"/>
+        <mass value="2e-06"/>
+        <inertia ixx="1.1e-09" ixy="0" ixz="0" iyy="1.1e-09" iyz="0" izz="1.1e-09"/>
+      </inertial>
+    </link>
+   <!-- Bottom Adapter- Electric Gripper Base joint -->
+    <joint name="${side}_electric_gripper_base_joint" type="fixed">
+	    <origin rpy="0 0 0" xyz="0 0 ${adapter_bottom_length}"/>
+      <parent link="${side}_adapter_bottom"/>
+      <child link="${side}_electric_gripper_base"/>
+    </joint>
+    <!-- Electric Gripper Base Link -->
+    <link name="${side}_electric_gripper_base">
+      <visual>
+	      <origin rpy="0 0 ${pi}" xyz="0 0 0"/>
+        <geometry>
+	<mesh filename="package://intera_tools_description/meshes/smart_pneumatic_gripper/gripper_base.STL" scale="0.001 0.001 0.001"/>
+        </geometry>
+      </visual>
+      <collision>
+	      <origin rpy="0 0 ${pi}" xyz="0 0 0"/>
+        <geometry>
+          <cylinder length="0.1" radius="0.029"/>
+        </geometry>
+        <material name="darkred">
+          <color rgba=".5 .1 .1 1"/>
+        </material>
+      </collision>
+      <inertial>
+        <origin rpy="0 0 0" xyz="0.0 0.0 0.0"/>
+        <mass value="2e-06"/>
+        <inertia ixx="1.1e-09" ixy="0" ixz="0" iyy="1.1e-09" iyz="0" izz="1.1e-09"/>
+      </inertial>
+    </link>
 <!-- Reference Joints, and links, non-visual, for transform references, and motion planning purposes -->
     <!--To connect this file with the sawyer_base.urdf.xacro a joint must be created between link "right_hand" in the latter file and "pneumatic_gripper_base", this way there is a transform between the robot last link and the End Of Arm Tooling in this file -->

Commit message: Smart pneumatic gripper URDF updated, visuals done

File: intera_tools_description/urdf/smart_pneumatic_gripper/rethink_pneumatic_gripper.xacro (robot description, xacro)
@@ -9,5 +9,5 @@
     <xacro:property name="end_of_arm_offset" value="-0.005" scope="local"/>
     <xacro:property name="connector_plate_length" value="0.032" scope="local"/>
-    <xacro:property name="pneumatic_gripper_base_length" value="0.04552" scope="local"/>
+    <xacro:property name="pneumatic_gripper_base_length" value="0.0282" scope="local"/>
     <xacro:property name="ft_sensor_length" value="0.033" scope="local"/>
     <xacro:property name="adapter_top_length" value="0.013" scope="local"/>
@@ -43,5 +43,5 @@
         <origin xyz="0 0 0" rpy="3.1416 0 0" />
         <geometry>
-		<mesh filename="package://intera_tools_description/meshes/smart_pneumatic_gripper/smart_click_adapter.STL" scale="0.001 0.001 0.001" />
+		<mesh filename="package://intera_tools_description/meshes/smart_pneumatic_gripper/STL/smart_click_adapter.STL" scale="0.001 0.001 0.001" />
         </geometry>
         <material name="black">
@@ -83,5 +83,5 @@
         <origin xyz="0 0 0" rpy="3.1416 0 0" />
         <geometry>
-		<mesh filename="package://intera_tools_description/meshes/smart_pneumatic_gripper/ati_9105_t_delta.STL" scale="0.001 0.001 0.001"/>
+		<mesh filename="package://intera_tools_description/meshes/smart_pneumatic_gripper/STL/ati_9105_t_delta.STL" scale="0.001 0.001 0.001"/>
         </geometry>
       </visual>
@@ -110,5 +110,5 @@
 	      <origin xyz="0 0 ${adapter_top_length}" rpy="${pi/2*-1} 0 0" />
         <geometry>
-		<mesh filename="package://intera_tools_description/meshes/smart_pneumatic_gripper/ft_gripper_adapter_top.STL" scale="0.001 0.001 0.001"/>
+		<mesh filename="package://intera_tools_description/meshes/smart_pneumatic_gripper/STL/ft_gripper_adapter_top.STL" scale="0.001 0.001 0.001"/>
         </geometry>
       </visual>
@@ -137,5 +137,5 @@
 	      <origin xyz="0 0 ${adapter_bottom_length}" rpy="${pi/2*-1} 0 0" />
         <geometry>
-		<mesh filename="package://intera_tools_description/meshes/smart_pneumatic_gripper/ft_gripper_adapter_bottom.STL" scale="0.001 0.001 0.001"/>
+		<mesh filename="package://intera_tools_description/meshes/smart_pneumatic_gripper/STL/ft_gripper_adapter_bottom.STL" scale="0.001 0.001 0.001"/>
         </geometry>
       </visual>
@@ -155,22 +155,28 @@
       </inertial>
     </link>
-   <!-- Bottom Adapter- Electric Gripper Base joint -->
-    <joint name="${side}_electric_gripper_base_joint" type="fixed">
+   <!-- Bottom Adapter- Pneumatic Gripper Base joint -->
+    <joint name="${side}_pneumatic_base_joint" type="fixed">
 	    <origin rpy="0 0 0" xyz="0 0 ${adapter_bottom_length}"/>
       <parent link="${side}_adapter_bottom"/>
-      <child link="${side}_electric_gripper_base"/>
-    </joint>
-    <!-- Electric Gripper Base Link -->
-    <link name="${side}_electric_gripper_base">
-      <visual>
-	      <origin rpy="0 0 ${pi}" xyz="0 0 0"/>
-        <geometry>
-	<mesh filename="package://intera_tools_description/meshes/smart_pneumatic_gripper/gripper_base.STL" scale="0.001 0.001 0.001"/>
-        </geometry>
-      </visual>
-      <collision>
-	      <origin rpy="0 0 ${pi}" xyz="0 0 0"/>
-        <geometry>
-          <cylinder length="0.1" radius="0.029"/>
+      <child link="${side}_pneumatic_gripper_base"/>
+    </joint>
+   <!-- Bottom Adapter- Pneumatic Gripper Cover joint -->
+    <joint name="${side}_pneumatic_cover_joint" type="fixed">
+	    <origin rpy="0 0 0" xyz="0 0 ${adapter_bottom_length}"/>
+      <parent link="${side}_adapter_bottom"/>
+      <child link="${side}_pneumatic_gripper_cover"/>
+    </joint>
+    <!-- Pneumatic Gripper Base Link (actuator) -->
+    <link name="${side}_pneumatic_gripper_base">
+      <visual>
+	      <origin rpy="${pi/2} 0 0" xyz="0 0 0"/>
+        <geometry>
+		<mesh filename="package://intera_tools_description/meshes/smart_pneumatic_gripper/STL/sz_16_base.STL" scale="0.001 0.001 0.001"/>
+        </geometry>
+      </visual>
+      <collision>
+	      <origin rpy="${pi/2} 0 0" xyz="0 0 0"/>
+        <geometry>
+          <cylinder length="0" radius="0"/>
         </geometry>
         <material name="darkred">
@@ -182,4 +188,255 @@
         <mass value="2e-06"/>
         <inertia ixx="1.1e-09" ixy="0" ixz="0" iyy="1.1e-09" iyz="0" izz="1.1e-09"/>
+      </inertial>
+    </link>
+    <!-- Pneumatic Gripper Cover -->
+    <link name="${side}_pneumatic_gripper_cover">
+      <visual>
+	      <origin rpy="0 0 ${pi}" xyz="0 0 0"/>
+        <geometry>
+		<mesh filename="package://intera_tools_description/meshes/smart_pneumatic_gripper/STL/gripper_base.STL" scale="0.001 0.001 0.001"/>
+        </geometry>
+      </visual>
+      <collision>
+	      <origin rpy="0 0 ${pi}" xyz="0 0 0"/>
+        <geometry>
+          <cylinder length="0.1" radius="0.029"/>
+        </geometry>
+        <material name="darkred">
+          <color rgba=".5 .1 .1 1"/>
+        </material>
+      </collision>
+    </link>
+    <!-- Left finger joint -->
+    <joint name="${side}_gripper_l_finger_joint" type="prismatic">
+      <origin rpy="0 0 0" xyz="0 0 ${pneumatic_gripper_base_length}"/>
+      <axis xyz="0 1 0"/>
+      <parent link="${side}_pneumatic_gripper_base"/>
+      <child link="${side}_gripper_l_finger"/>
+      <limit effort="20.0" lower="0.0" upper="0.016" velocity="5.0"/>
+      <dynamics damping="100.0" friction="500.0"/>
+    </joint>
+    <!-- Left finger gripper base link -->
+   <link name="${side}_gripper_l_finger">
+      <visual>
+	      <origin rpy="${pi/2} 0 0" xyz="0 0.0295 0"/>
+        <geometry>
+	<mesh filename="package://intera_tools_description/meshes/smart_pneumatic_gripper/STL/sz_16_finger.STL" scale="0.001 0.001 0.001"/>
+        </geometry>
+      </visual>
+      <collision>
+	      <origin rpy="${pi/2} 0 0" xyz="0 0.0295 0"/>
+        <geometry>
+          <box size="0 0 0"/>
+        </geometry>
+      </collision>
+      <inertial>
+        <origin rpy="0 0 0" xyz="0 0 0"/>
+        <mass value="0.001"/>
+        <inertia ixx="0.01" ixy="0" ixz="0" iyy="0.01" iyz="0" izz="0.01"/>
+      </inertial>
+    </link>
+    <xacro:if value="${gazebo}">
+      <gazebo reference="${side}_gripper_l_finger">
+        <mu1>1000</mu1>
+        <mu2>1000</mu2>
+        <fdir1>0.0 0.0 1.0</fdir1>
+        <kp>1e5</kp>
+        <kd>1.0</kd>
+      </gazebo>
+    </xacro:if>
+    <!-- Left finger gripper base - finger base joint -->
+    <joint name="${side}_gripper_l_finger_base_joint" type="fixed">
+	    <origin rpy="0 0 0" xyz="0 0 0.012"/>
+      <parent link="${side}_gripper_l_finger"/>
+      <child link="${side}_gripper_l_finger_base"/>
+    </joint>
+    <!-- Left finger base link -->
+   <link name="${side}_gripper_l_finger_base">
+      <visual>
+	      <origin rpy="0 0 ${pi/2}" xyz="0 0.0185 0"/>
+        <geometry>
+        <mesh filename="package://intera_tools_description/meshes/smart_pneumatic_gripper/STL/pneumatic_finger_base.STL" scale="0.001 0.001 0.001"/>
+        </geometry>
+      </visual>
+      <collision>
+	      <origin rpy="0 0 ${pi/2}" xyz="0 0.0185 0"/>
+        <geometry>
+          <box size="0 0 0"/>
+        </geometry>
+      </collision>
+      <inertial>
+        <origin rpy="0 0 0" xyz="0 0 0"/>
+        <mass value="0.001"/>
+        <inertia ixx="0.01" ixy="0" ixz="0" iyy="0.01" iyz="0" izz="0.01"/>
+      </inertial>
+    </link>
+    <!-- Left finger base - finger body joint -->
+    <joint name="${side}_gripper_l_finger_body_joint" type="fixed">
+	    <origin rpy="0 0 0" xyz="0 0 0.006"/>
+      <parent link="${side}_gripper_l_finger_base"/>
+      <child link="${side}_gripper_l_finger_body"/>
+    </joint>
+    <!-- Left finger body link -->
+   <link name="${side}_gripper_l_finger_body">
+      <visual>
+	      <origin rpy="0 0 ${pi/2}" xyz="0 0.021 0"/>
+        <geometry>
+        <mesh filename="package://intera_tools_description/meshes/smart_pneumatic_gripper/STL/pneumatic_finger.STL" scale="0.001 0.001 0.001"/>
+        </geometry>
+      </visual>
+      <collision>
+	      <origin rpy="0 0 ${pi/2}" xyz="0 0.021 0"/>
+        <geometry>
+          <box size="0 0 0"/>
+        </geometry>
+      </collision>
+      <inertial>
+        <origin rpy="0 0 0" xyz="0 0 0"/>
+        <mass value="0.001"/>
+        <inertia ixx="0.01" ixy="0" ixz="0" iyy="0.01" iyz="0" izz="0.01"/>
+      </inertial>
+    </link>
+    <!-- Left finger body - finger tip joint -->
+    <joint name="${side}_gripper_l_finger_tip_joint" type="fixed">
+	    <origin rpy="0 0 0" xyz="0 0 0"/>
+      <parent link="${side}_gripper_l_finger_body"/>
+      <child link="${side}_gripper_l_finger_tip"/>
+    </joint>
+    <!-- Left finger tip link -->
+   <link name="${side}_gripper_l_finger_tip">
+      <visual>
+	      <origin rpy="0 0 ${pi/2}" xyz="0 0.021 0.0726"/>
+        <geometry>
+        <mesh filename="package://intera_tools_description/meshes/smart_pneumatic_gripper/STL/pneumatic_finger_tip.STL" scale="0.001 0.001 0.001"/>
+        </geometry>
+      </visual>
+      <collision>
+	      <origin rpy="0 0 ${pi/2}" xyz="0 0.021 0.0726"/>
+        <geometry>
+          <box size="0 0 0"/>
+        </geometry>
+      </collision>
+      <inertial>
+        <origin rpy="0 0 0" xyz="0 0 0"/>
+        <mass value="0.001"/>
+        <inertia ixx="0.01" ixy="0" ixz="0" iyy="0.01" iyz="0" izz="0.01"/>
+      </inertial>
+    </link>
+    <!-- Right finger joint -->
+    <joint name="${side}_gripper_r_finger_joint" type="prismatic">
+      <origin rpy="0 0 0" xyz="0 0 ${pneumatic_gripper_base_length}"/>
+      <axis xyz="0 1 0"/>
+      <parent link="${side}_pneumatic_gripper_base"/>
+      <child link="${side}_gripper_r_finger"/>
+      <limit effort="20.0" lower="-0.016" upper="0.0" velocity="5.0"/>
+      <mimic joint="${side}_gripper_l_finger_joint" multiplier="-1.0"/>
+      <dynamics damping="100.0" friction="500.0"/>
+    </joint>
+    <!-- Right finger gripper base link -->
+   <link name="${side}_gripper_r_finger">
+      <visual>
+	      <origin rpy="${pi/2} 0 ${pi}" xyz="0 -0.0295 0"/>
+        <geometry>
+	<mesh filename="package://intera_tools_description/meshes/smart_pneumatic_gripper/STL/sz_16_finger.STL" scale="0.001 0.001 0.001"/>
+        </geometry>
+      </visual>
+      <collision>
+	      <origin rpy="${pi/2} 0 ${pi}" xyz="0 -0.0295 0"/>
+        <geometry>
+          <box size="0 0 0"/>
+        </geometry>
+      </collision>
+      <inertial>
+        <origin rpy="0 0 0" xyz="0 0 0"/>
+        <mass value="0.001"/>
+        <inertia ixx="0.01" ixy="0" ixz="0" iyy="0.01" iyz="0" izz="0.01"/>
+      </inertial>
+    </link>
+    <xacro:if value="${gazebo}">
+      <gazebo reference="${side}_gripper_r_finger">
+        <mu1>1000</mu1>
+        <mu2>1000</mu2>
+        <fdir1>0.0 0.0 1.0</fdir1>
+        <kp>1e5</kp>
+        <kd>1.0</kd>
+      </gazebo>
+    </xacro:if>
+    <!-- Right finger gripper base - finger base joint -->
+    <joint name="${side}_gripper_r_finger_base_joint" type="fixed">
+	    <origin rpy="0 0 0" xyz="0 0 0.012"/>
+      <parent link="${side}_gripper_r_finger"/>
+      <child link="${side}_gripper_r_finger_base"/>
+    </joint>
+    <!-- Right finger base link -->
+   <link name="${side}_gripper_r_finger_base">
+      <visual>
+	      <origin rpy="0 0 ${-pi/2}" xyz="0 -0.0185 0"/>
+        <geometry>
+        <mesh filename="package://intera_tools_description/meshes/smart_pneumatic_gripper/STL/pneumatic_finger_base.STL" scale="0.001 0.001 0.001"/>
+        </geometry>
+      </visual>
+      <collision>
+	      <origin rpy="0 0 ${-pi/2}" xyz="0 -0.0185 0"/>
+        <geometry>
+          <box size="0 0 0"/>
+        </geometry>
+      </collision>
+      <inertial>
+        <origin rpy="0 0 0" xyz="0 0 0"/>
+        <mass value="0.001"/>
+        <inertia ixx="0.01" ixy="0" ixz="0" iyy="0.01" iyz="0" izz="0.01"/>
+      </inertial>
+    </link>
+    <!-- Right finger base - finger body joint -->
+    <joint name="${side}_gripper_r_finger_body_joint" type="fixed">
+	    <origin rpy="0 0 0" xyz="0 0 0.006"/>
+      <parent link="${side}_gripper_r_finger_base"/>
+      <child link="${side}_gripper_r_finger_body"/>
+    </joint>
+    <!-- Right finger body link -->
+   <link name="${side}_gripper_r_finger_body">
+      <visual>
+	      <origin rpy="0 0 ${-pi/2}" xyz="0 -0.021 0"/>
+        <geometry>
+        <mesh filename="package://intera_tools_description/meshes/smart_pneumatic_gripper/STL/pneumatic_finger.STL" scale="0.001 0.001 0.001"/>
+        </geometry>
+      </visual>
+      <collision>
+	      <origin rpy="0 0 ${-pi/2}" xyz="0 -0.021 0"/>
+        <geometry>
+          <box size="0 0 0"/>
+        </geometry>
+      </collision>
+      <inertial>
+        <origin rpy="0 0 0" xyz="0 0 0"/>
+        <mass value="0.001"/>
+        <inertia ixx="0.01" ixy="0" ixz="0" iyy="0.01" iyz="0" izz="0.01"/>
+      </inertial>
+    </link>
+    <!-- Right finger body - finger tip joint -->
+    <joint name="${side}_gripper_r_finger_tip_joint" type="fixed">
+	    <origin rpy="0 0 0" xyz="0 0 0"/>
+      <parent link="${side}_gripper_r_finger_body"/>
+      <child link="${side}_gripper_r_finger_tip"/>
+    </joint>
+    <!-- Right finger tip link -->
+   <link name="${side}_gripper_r_finger_tip">
+      <visual>
+	      <origin rpy="0 0 ${-pi/2}" xyz="0 -0.021 0.0726"/>
+        <geometry>
+        <mesh filename="package://intera_tools_description/meshes/smart_pneumatic_gripper/STL/pneumatic_finger_tip.STL" scale="0.001 0.001 0.001"/>
+        </geometry>
+      </visual>
+      <collision>
+	      <origin rpy="0 0 ${-pi/2}" xyz="0 -0.021 0.0726"/>
+        <geometry>
+          <box size="0 0 0"/>
+        </geometry>
+      </collision>
+      <inertial>
+        <origin rpy="0 0 0" xyz="0 0 0"/>
+        <mass value="0.001"/>
+        <inertia ixx="0.01" ixy="0" ixz="0" iyy="0.01" iyz="0" izz="0.01"/>
       </inertial>
     </link>
@@ -209,4 +466,33 @@
       </inertial>
     </link>
+    <!-- Gazebo References -->
+        <xacro:if value="${gazebo}">
+    <transmission name="gripper_${side}1">
+      <type>transmission_interface/SimpleTransmission</type>
+      <joint name="${side}_gripper_r_finger_joint">
+        <hardwareInterface>hardware_interface/EffortJointInterface</hardwareInterface>
+      </joint>
+      <actuator name="gripper_${side}1_motor1">
+        <hardwareInterface>hardware_interface/EffortJointInterface</hardwareInterface>
+        <mechanicalReduction>1</mechanicalReduction>
+      </actuator>
+    </transmission>
+    <transmission name="gripper_${side}2">
+      <type>transmission_interface/SimpleTransmission</type>
+      <joint name="${side}_gripper_l_finger_joint">
+        <hardwareInterface>hardware_interface/EffortJointInterface</hardwareInterface>
+      </joint>
+      <actuator name="gripper_${side}1_motor2">
+        <hardwareInterface>hardware_interface/EffortJointInterface</hardwareInterface>
+        <mechanicalReduction>1</mechanicalReduction>
+      </actuator>
+    </transmission>
+    <gazebo reference="${side}_gripper_r_finger_joint">
+      <implicitSpringDamper>1</implicitSpringDamper>
+    </gazebo>
+    <gazebo reference="${side}_gripper_l_finger_joint">
+      <implicitSpringDamper>1</implicitSpringDamper>
+    </gazebo>
+    </xacro:if>
   </xacro:macro>
 </robot>
