Commit message: Smart pneumatic gripper updated, slot position feature added, collision, lenghts and tip length updated

File: intera_tools_description/urdf/smart_pneumatic_gripper/rethink_pneumatic_gripper.xacro (robot description, xacro)
@@ -16,5 +16,9 @@
     <xacro:property name="adapter_top_length" value="0.013" scope="local"/>
     <xacro:property name="adapter_bottom_length" value="0.018" scope="local"/>
-    <xacro:property name="finger_length" value="0.0021" scope="local"/>
+<!-- Finger Length Properties -->
+    <xacro:property name="finger_move_length" value="0.012" scope="local"/>
+    <xacro:property name="finger_base_length" value="0.006" scope="local"/>
+    <xacro:property name="finger_to_tip_length" value="${0.0726-((tip_slot_pos-1)*0.015)}" scope="local"/>
+    <xacro:property name="finger_total_length" value="${finger_move_length + finger_base_length + finger_to_tip_length}" scope="local"/>
 <!-- Start Kinematic Chain -->
 <!-- Structure is ordered as a tree: link, joint, link, to observe geometrical relationships between each of them-->
@@ -112,5 +116,11 @@
     <joint name="${side}_ft_sensor_adapter_top_joint" type="fixed">        <origin xyz="0 0 ${ft_sensor_length}" rpy="0 0 0" />                 <parent link="${side}_ft_sensor_link" />
       <child  link="${side}_adapter_top" />
-    </joint>
+      <provideFeedback>true</provideFeedback>
+    </joint>
+        <plugin name="ft_sensor" filename="libgazebo_ros_ft_sensor.so">
+            <updateRate>100.0</updateRate>
+            <topicName>ft_sensor_topic</topicName>
+            <jointName>${side}_ft_sensor_adapter_top_joint</jointName>
+        </plugin>
     <!-- Adapter Top Part Link -->
     <link name="${side}_adapter_top">
@@ -284,5 +294,5 @@
       </visual>
       <collision>
-	      <origin rpy="0 0 ${pi/2}" xyz="0 0.061 0"/>
+	      <origin rpy="0 0 ${pi/2}" xyz="0 0.047 0.003"/>
         <geometry>
           <box size="0.085 0.024 0.006"/>
@@ -300,5 +310,5 @@
     <!-- Left finger base - finger body joint -->
     <joint name="${side}_gripper_l_finger_body_joint" type="fixed">
-	    <origin rpy="0 0 0" xyz="0 0 0.006"/>
+	    <origin rpy="0 0 0" xyz="0 ${(finger_slot_pos-1)*0.008} 0.006"/>
       <parent link="${side}_gripper_l_finger_base"/>
       <child link="${side}_gripper_l_finger_body"/>
@@ -307,5 +317,5 @@
    <link name="${side}_gripper_l_finger_body">
       <visual>
-	      <origin rpy="0 0 ${pi/2}" xyz="0 0.021 0"/>
+	      <origin rpy="0 0 ${pi/2}" xyz="0 -0.0035 0"/>
         <geometry>
         <mesh filename="package://intera_tools_description/meshes/smart_pneumatic_gripper/STL/pneumatic_finger.STL" scale="0.001 0.001 0.001"/>
@@ -313,5 +323,5 @@
       </visual>
       <collision>
-	  <origin rpy="0 0 0" xyz="0 0.024 0.04475"/>
+	  <origin rpy="0 0 0" xyz="0 -0.0005 0.03975"/>
         <geometry>
           <box size="0.0275 0.006 0.0795"/>
@@ -322,5 +332,5 @@
       </collision>
       <inertial>
-	<origin rpy="0 0 ${pi/2}" xyz="0 0.021 0"/>
+	<origin rpy="0 0 ${pi/2}" xyz="0 -0.0035 0"/>
         <mass value="0.001"/>
         <inertia ixx="0.0000683111" ixy="-1.24623E-9" ixz="0.0000038251" iyy="0.0000668321" iyz="-1.738481E-8" izz="0.0000031831"/>
@@ -336,5 +346,5 @@
    <link name="${side}_gripper_l_finger_tip">
       <visual>
-	      <origin rpy="0 0 ${pi/2}" xyz="0 0.021 0.0726"/>
+	      <origin rpy="0 0 ${pi/2}" xyz="0 -0.0035 ${0.0726-((tip_slot_pos-1)*0.015)}"/>
         <geometry>
         <mesh filename="package://intera_tools_description/meshes/smart_pneumatic_gripper/STL/pneumatic_finger_tip.STL" scale="0.001 0.001 0.001"/>
@@ -342,5 +352,5 @@
       </visual>
       <collision>
-	      <origin rpy="0 0 ${pi/2}" xyz="0 0.021 0.0726"/>
+	      <origin rpy="0 0 ${pi/2}" xyz="0 -0.0035 ${0.0726-((tip_slot_pos-1)*0.015)}"/>
         <geometry>
               <mesh filename="package://intera_tools_description/meshes/smart_pneumatic_gripper/STL/pneumatic_finger_tip.STL" scale="0.001 0.001 0.001"/>
@@ -351,5 +361,5 @@
       </collision>
       <inertial>
-	      <origin rpy="0 0 ${pi/2}" xyz="0 0.021 0.0726"/>
+	      <origin rpy="0 0 ${pi/2}" xyz="0 -0.0035 ${0.0726-((tip_slot_pos-1)*0.015)}"/>
         <mass value="0.001"/>
         <inertia ixx="0.0000064492" ixy="-2.802891E-8" ixz="-2.65457E-9" iyy="0.0000019488" iyz="1.4972E-10" izz="0.0000057675"/>
@@ -411,5 +421,5 @@
       </visual>
       <collision>
-              <origin rpy="0 0 ${-pi/2}" xyz="0 -0.061 0"/>
+              <origin rpy="0 0 ${-pi/2}" xyz="0 -0.047 0.003"/>
         <geometry>
           <box size="0.085 0.024 0.006"/>
@@ -427,5 +437,5 @@
     <!-- Right finger base - finger body joint -->
     <joint name="${side}_gripper_r_finger_body_joint" type="fixed">
-	    <origin rpy="0 0 0" xyz="0 0 0.006"/>
+	    <origin rpy="0 0 0" xyz="0 ${(finger_slot_pos-1)*-0.008} 0.006"/>
       <parent link="${side}_gripper_r_finger_base"/>
       <child link="${side}_gripper_r_finger_body"/>
@@ -434,5 +444,5 @@
    <link name="${side}_gripper_r_finger_body">
       <visual>
-	      <origin rpy="0 0 ${-pi/2}" xyz="0 -0.021 0"/>
+	      <origin rpy="0 0 ${-pi/2}" xyz="0 0.0035 0"/>
         <geometry>
         <mesh filename="package://intera_tools_description/meshes/smart_pneumatic_gripper/STL/pneumatic_finger.STL" scale="0.001 0.001 0.001"/>
@@ -440,5 +450,5 @@
       </visual>
       <collision>
-          <origin rpy="0 0 0" xyz="0 -0.024 0.04475"/>
+          <origin rpy="0 0 0" xyz="0 0.0005 0.03975"/>
         <geometry>
           <box size="0.0275 0.006 0.0795"/>
@@ -449,5 +459,5 @@
       </collision>
       <inertial>
-	      <origin rpy="0 0 ${-pi/2}" xyz="0 -0.021 0"/>
+	      <origin rpy="0 0 ${-pi/2}" xyz="0 0.0035 0"/>
         <mass value="0.001"/>
         <inertia ixx="0.0000683111" ixy="-1.24623E-9" ixz="0.0000038251" iyy="0.0000668321" iyz="-1.738481E-8" izz="0.0000031831"/>
@@ -463,5 +473,5 @@
    <link name="${side}_gripper_r_finger_tip">
       <visual>
-	      <origin rpy="0 0 ${-pi/2}" xyz="0 -0.021 0.0726"/>
+	      <origin rpy="0 0 ${-pi/2}" xyz="0 0.0035 ${0.0726-((tip_slot_pos-1)*0.015)}"/>
         <geometry>
         <mesh filename="package://intera_tools_description/meshes/smart_pneumatic_gripper/STL/pneumatic_finger_tip.STL" scale="0.001 0.001 0.001"/>
@@ -469,5 +479,5 @@
       </visual>
       <collision>
-              <origin rpy="0 0 ${-pi/2}" xyz="0 -0.021 0.0726"/>
+              <origin rpy="0 0 ${-pi/2}" xyz="0 0.0035 ${0.0726-((tip_slot_pos-1)*0.015)}"/>
         <geometry>
               <mesh filename="package://intera_tools_description/meshes/smart_pneumatic_gripper/STL/pneumatic_finger_tip.STL" scale="0.001 0.001 0.001"/>
@@ -478,5 +488,5 @@
       </collision>
       <inertial>
-	      <origin rpy="0 0 ${-pi/2}" xyz="0 -0.021 0.0726"/>
+	      <origin rpy="0 0 ${-pi/2}" xyz="0 0.0035 ${0.0726-((tip_slot_pos-1)*0.015)}"/>
         <mass value="0.001"/>
         <inertia ixx="0.0000064492" ixy="-2.802891E-8" ixz="-2.65457E-9" iyy="0.0000019488" iyz="1.4972E-10" izz="0.0000057675"/>
@@ -487,6 +497,6 @@
     <!-- Gripper Base Joint -->
     <!-- "right_hand" link position is with respect to its correponding joint, so the end_of_arm_offset is with respect to the last joint at the robot end effector at sawyer_base.urdf.xacro -->
-    <xacro:property name="end_of_arm_offset" value="-0.005" scope="local"/>
-    <joint name="${side}_gripper_base_joint" type="fixed">						  <origin rpy="0 0 0" xyz="0 0 ${end_of_arm_offset}"/>
+    <joint name="${side}_gripper_base_joint" type="fixed">
+      <origin rpy="0 0 0" xyz="0 0 ${end_of_arm_offset}"/>
       <parent link="${side}_hand"/>
       <child link="${side}_gripper_base"/>
@@ -495,5 +505,5 @@
     <!-- Gripper Tip joint -->
     <joint name="${side}_gripper_tip_joint" type="fixed">
-      <origin rpy="0 0 0" xyz="0 0 ${(-1*end_of_arm_offset)+connector_plate_length+pneumatic_gripper_base_length+finger_length}"/>
+      <origin rpy="0 0 0" xyz="0 0 ${connector_plate_length+ft_sensor_length+adapter_top_length+adapter_bottom_length+pneumatic_gripper_base_length+finger_total_length}"/>
       <parent link="${side}_gripper_base"/>
       <child link="${side}_gripper_tip"/>

Commit message: Smart pneumatic gripper updated, link mass updated, finger tip lenght updated, F/T sensor added topic publishing but no force measurement adquired

File: intera_tools_description/urdf/smart_pneumatic_gripper/rethink_pneumatic_gripper.xacro (robot description, xacro)
@@ -8,5 +8,5 @@
 <!-- Lenght Properties of each element in End of Arm Tooling -->
 <!-- #ToDo Update distances in meters for pneumatic gripper -->
-    <xacro:property name="end_of_arm_offset" value="-0.012" scope="local"/>
+    <xacro:property name="end_of_arm_offset" value="-0.009" scope="local"/>
     <xacro:property name="tip_slot_offset" value="0.015" scope="local"/>
     <xacro:property name="finger_slot_offset" value="-0.008" scope="local"/>
@@ -28,5 +28,5 @@
       <inertial>
         <!-- Sum Gripper Mass - for whole end effector, measured from end of plastic cuff -->
-        <mass value="0.47"/>
+        <mass value="1.902"/>
         <origin rpy="0 0 0" xyz="0.0028 -0.0004 0.0343"/>
         <inertia ixx="1e-08" ixy="0" ixz="0" iyy="1e-08" iyz="0" izz="1e-08"/>
@@ -43,5 +43,5 @@
       <inertial>
 	      <origin xyz="0 0 0" rpy="${pi} 0 0" />
-        <mass value="0.0" />
+        <mass value="0.387" />
         <inertia ixx="0.0000292897"  ixy="6.1026E-08"  ixz="-1.5353186E-7"
                iyy="0.0000296079"  iyz="-3.597884E-8" izz="0.0000508198" />
@@ -88,5 +88,5 @@
     <link name="${side}_ft_sensor_link">
       <visual>
-	<origin xyz="0 0 0" rpy="${pi} 0 0" />
+	      <origin xyz="0 0 0" rpy="${pi} 0 ${pi/2}" />
         <geometry>
 		<mesh filename="package://intera_tools_description/meshes/smart_pneumatic_gripper/STL/ati_9105_t_delta.STL" scale="0.001 0.001 0.001"/>
@@ -94,5 +94,5 @@
       </visual>
       <collision>
-	      <origin xyz="0 0 ${ft_sensor_length*0.5}" rpy="${pi} 0 0" />
+	      <origin xyz="0 0 ${ft_sensor_length*0.5}" rpy="${pi} 0 ${pi/2}" />
         <geometry>
 		<cylinder length="${ft_sensor_length}" radius="0.046"/>
@@ -103,6 +103,6 @@
       </collision>
       <inertial>
-	<origin rpy="${pi} 0 0" xyz="0 0 0"/>
-        <mass value="2e-06"/>
+	      <origin rpy="${pi} 0 ${pi/2}" xyz="0 0 0"/>
+        <mass value="0.919"/>
         <inertia ixx="0.0001756735" ixy="6.8322E-8" ixz="-2.7814E-8" iyy="0.0001757811" iyz="-9.2588E-8" izz="0.0002122946"/>
       </inertial>
@@ -116,11 +116,29 @@
     <joint name="${side}_ft_sensor_adapter_top_joint" type="fixed">        <origin xyz="0 0 ${ft_sensor_length}" rpy="0 0 0" />                 <parent link="${side}_ft_sensor_link" />
       <child  link="${side}_adapter_top" />
-      <provideFeedback>true</provideFeedback>
-    </joint>
-        <plugin name="ft_sensor" filename="libgazebo_ros_ft_sensor.so">
-            <updateRate>100.0</updateRate>
-            <topicName>ft_sensor_topic</topicName>
-            <jointName>${side}_ft_sensor_adapter_top_joint</jointName>
-        </plugin>
+    </joint>
+    <!-- Fixed joint from F/T to tip to measure forces at the end effector -->
+    <joint name="${side}_ft_sensor_tip_joint" type="revolute">
+	    <origin xyz="0 0 ${ft_sensor_length}" rpy="0 0 ${pi/2}" />
+      <parent link="${side}_ft_sensor_link"  />
+      <child  link="${side}_ft_measure_tip" />
+      <limit lower="0" upper="0" effort="1000" velocity="6.5"/>
+    </joint>
+    <gazebo reference="${side}_ft_sensor_tip_joint">
+    	<provideFeedback>true</provideFeedback>
+    </gazebo>
+<gazebo>
+  <plugin name="gazebo_ros_ft_sensor" filename="libgazebo_ros_ft_sensor.so">
+    <!-- Required parameters -->
+    <updateRate>100.0</updateRate>
+    <always_on>true</always_on>
+    <visualize>true</visualize>
+    <jointName>${side}_ft_sensor_tip_joint</jointName>
+    <topicName>/robot/ft_sensor_topic</topicName>
+    <force_torque>
+    	<frame>sensor</frame>
+    	<measure_direction>parent_to_child</measure_direction>
+    </force_torque>
+  </plugin>
+</gazebo>
     <!-- Adapter Top Part Link -->
     <link name="${side}_adapter_top">
@@ -142,5 +160,5 @@
       <inertial>
         <origin rpy="${-pi/2} 0 0" xyz="0.0 0.0 0.0"/>
-        <mass value="2e-06"/>
+        <mass value="0.061"/>
         <inertia ixx="0.0000418848" ixy="0" ixz="0" iyy="0.0000761051" iyz="0" izz="0.0000418848"/>
       </inertial>
@@ -174,5 +192,5 @@
       <inertial>
 	<origin rpy="${-pi/2} 0 ${pi/2}" xyz="0.0 0.0 0.0"/>
-        <mass value="2e-06"/>
+        <mass value="0.098"/>
         <inertia ixx="0.0000721906" ixy="0" ixz="0" iyy="0.0001202265" iyz="0" izz="0.0000723151"/>
       </inertial>
@@ -214,5 +232,5 @@
       <inertial>
 	      <origin rpy="${pi/2} 0 0" xyz="0.0 0.0 0.0"/>
-        <mass value="2e-06"/>
+        <mass value="0.311"/>
         <inertia ixx="0.0000330475" ixy="1.31E-8" ixz="0" iyy="0.0000176978" iyz="0" izz="0.0000203961"/>
       </inertial>
@@ -265,5 +283,5 @@
       <inertial>
 	<origin rpy="${pi/2} 0 0" xyz="0 0.0295 0"/>
-        <mass value="0.001"/>
+        <mass value="0.010"/>
         <inertia ixx="0.0000013187" ixy="0" ixz="0" iyy="0.0000012511" iyz="2.8731E-7" izz="2.2756E-7"/>
       </inertial>
@@ -304,5 +322,5 @@
       <inertial>
 	      <origin rpy="0 0 ${pi/2}" xyz="0 0.0185 0"/>
-        <mass value="0.001"/>
+        <mass value="0.029"/>
         <inertia ixx="0.00000151" ixy="-1.23E-12" ixz="0.0000025354" iyy="0.000042463" iyz="-1.23E-12" izz="0.0000433196"/>
       </inertial>
@@ -333,5 +351,5 @@
       <inertial>
 	<origin rpy="0 0 ${pi/2}" xyz="0 -0.0035 0"/>
-        <mass value="0.001"/>
+        <mass value="0.037"/>
         <inertia ixx="0.0000683111" ixy="-1.24623E-9" ixz="0.0000038251" iyy="0.0000668321" iyz="-1.738481E-8" izz="0.0000031831"/>
       </inertial>
@@ -362,5 +380,5 @@
       <inertial>
 	      <origin rpy="0 0 ${pi/2}" xyz="0 -0.0035 ${0.0726-((tip_slot_pos-1)*0.015)}"/>
-        <mass value="0.001"/>
+        <mass value="0.040"/>
         <inertia ixx="0.0000064492" ixy="-2.802891E-8" ixz="-2.65457E-9" iyy="0.0000019488" iyz="1.4972E-10" izz="0.0000057675"/>
       </inertial>
@@ -392,5 +410,5 @@
       <inertial>
 	      <origin rpy="${pi/2} 0 ${pi}" xyz="0 -0.0295 0"/>
-        <mass value="0.001"/>
+        <mass value="0.010"/>
         <inertia ixx="0.0000013187" ixy="0" ixz="0" iyy="0.0000012511" iyz="2.8731E-7" izz="2.2756E-7"/>
       </inertial>
@@ -431,5 +449,5 @@
       <inertial>
 	      <origin rpy="0 0 ${-pi/2}" xyz="0 -0.0185 0"/>
-        <mass value="0.001"/>
+        <mass value="0.029"/>
         <inertia ixx="0.00000151" ixy="-1.23E-12" ixz="0.0000025354" iyy="0.000042463" iyz="-1.23E-12" izz="0.0000433196"/>
       </inertial>
@@ -460,5 +478,5 @@
       <inertial>
 	      <origin rpy="0 0 ${-pi/2}" xyz="0 0.0035 0"/>
-        <mass value="0.001"/>
+        <mass value="0.037"/>
         <inertia ixx="0.0000683111" ixy="-1.24623E-9" ixz="0.0000038251" iyy="0.0000668321" iyz="-1.738481E-8" izz="0.0000031831"/>
       </inertial>
@@ -489,5 +507,5 @@
       <inertial>
 	      <origin rpy="0 0 ${-pi/2}" xyz="0 0.0035 ${0.0726-((tip_slot_pos-1)*0.015)}"/>
-        <mass value="0.001"/>
+        <mass value="0.040"/>
         <inertia ixx="0.0000064492" ixy="-2.802891E-8" ixz="-2.65457E-9" iyy="0.0000019488" iyz="1.4972E-10" izz="0.0000057675"/>
       </inertial>
@@ -505,10 +523,18 @@
     <!-- Gripper Tip joint -->
     <joint name="${side}_gripper_tip_joint" type="fixed">
-      <origin rpy="0 0 0" xyz="0 0 ${connector_plate_length+ft_sensor_length+adapter_top_length+adapter_bottom_length+pneumatic_gripper_base_length+finger_total_length}"/>
+      <origin rpy="0 0 0" xyz="0 0 ${(end_of_arm_offset*-1)+connector_plate_length+ft_sensor_length+adapter_top_length+adapter_bottom_length+pneumatic_gripper_base_length+finger_total_length}"/>
       <parent link="${side}_gripper_base"/>
       <child link="${side}_gripper_tip"/>
     </joint>
-    <!-- Electric Gripper Tip link -->
+    <!-- Pneumatic Gripper Tip link -->
     <link name="${side}_gripper_tip">
+      <inertial>
+        <origin xyz="0 0 0" rpy="0 0 0"/>
+        <mass value="2e-06"/>
+        <inertia ixx="1.1e-09" ixy="0" ixz="0" iyy="1.1e-09" iyz="0" izz="1.1e-09"/>
+      </inertial>
+    </link>
+    <!-- F/T sensor measure point at Tip link -->
+    <link name="${side}_ft_measure_tip">
       <inertial>
         <origin xyz="0 0 0" rpy="0 0 0"/>

Commit message: F/T Sensor in smart pneumatic gripper updated

File: intera_tools_description/urdf/smart_pneumatic_gripper/rethink_pneumatic_gripper.xacro (robot description, xacro)
@@ -119,8 +119,9 @@
     <!-- Fixed joint from F/T to tip to measure forces at the end effector -->
     <joint name="${side}_ft_sensor_tip_joint" type="revolute">
-	    <origin xyz="0 0 ${ft_sensor_length}" rpy="0 0 ${pi/2}" />
+      <origin xyz="0 0 ${ft_sensor_length+adapter_top_length+adapter_bottom_length+pneumatic_gripper_base_length+finger_total_length}" rpy="0 0 0" />
+      <axis xyz="1 0 0"/>
       <parent link="${side}_ft_sensor_link"  />
       <child  link="${side}_ft_measure_tip" />
-      <limit lower="0" upper="0" effort="1000" velocity="6.5"/>
+      <limit lower="-0.001" upper="0.001" effort="1000" velocity="1000"/>
     </joint>
     <gazebo reference="${side}_ft_sensor_tip_joint">
@@ -136,5 +137,5 @@
     <topicName>/robot/ft_sensor_topic</topicName>
     <force_torque>
-    	<frame>sensor</frame>
+    	<frame>parent</frame>
     	<measure_direction>parent_to_child</measure_direction>
     </force_torque>
@@ -537,4 +538,10 @@
     <!-- F/T sensor measure point at Tip link -->
     <link name="${side}_ft_measure_tip">
+       <visual>
+              <origin rpy="0 0 0" xyz="0 0 0"/>
+        <geometry>
+          <box size="0.00001 0.00001 0.00001"/>
+        </geometry>
+      </visual>
       <inertial>
         <origin xyz="0 0 0" rpy="0 0 0"/>

Commit message: F/T sensor for smart_pneumatic_gripper reference joint updated

File: intera_tools_description/urdf/smart_pneumatic_gripper/rethink_pneumatic_gripper.xacro (robot description, xacro)
@@ -114,16 +114,10 @@
     </xacro:if>
     <!-- F/T Sensor-Adapter Top Part Joint -->
-    <joint name="${side}_ft_sensor_adapter_top_joint" type="fixed">        <origin xyz="0 0 ${ft_sensor_length}" rpy="0 0 0" />                 <parent link="${side}_ft_sensor_link" />
-      <child  link="${side}_adapter_top" />
-    </joint>
-    <!-- Fixed joint from F/T to tip to measure forces at the end effector -->
-    <joint name="${side}_ft_sensor_tip_joint" type="revolute">
-      <origin xyz="0 0 ${ft_sensor_length+adapter_top_length+adapter_bottom_length+pneumatic_gripper_base_length+finger_total_length}" rpy="0 0 0" />
-      <axis xyz="1 0 0"/>
-      <parent link="${side}_ft_sensor_link"  />
-      <child  link="${side}_ft_measure_tip" />
-      <limit lower="-0.001" upper="0.001" effort="1000" velocity="1000"/>
-    </joint>
-    <gazebo reference="${side}_ft_sensor_tip_joint">
+    <joint name="${side}_ft_sensor_adapter_top_joint" type="revolute">                                       <origin xyz="0 0 ${ft_sensor_length}" rpy="0 0 0" />                                                <parent link="${side}_ft_sensor_link" />
+         <child  link="${side}_adapter_top" />
+         <axis xyz="1 0 0"/>
+         <limit lower="-0.001" upper="0.001" effort="1000" velocity="1000"/>
+    </joint>
+    <gazebo reference="${side}_ft_sensor_adapter_top_joint">
     	<provideFeedback>true</provideFeedback>
     </gazebo>
@@ -133,10 +127,9 @@
     <updateRate>100.0</updateRate>
     <always_on>true</always_on>
-    <visualize>true</visualize>
-    <jointName>${side}_ft_sensor_tip_joint</jointName>
+    <pose>0 0 0 3.1416 0 1.570759</pose>
+    <jointName>${side}_ft_sensor_adapter_top_joint</jointName>
     <topicName>/robot/ft_sensor_topic</topicName>
     <force_torque>
-    	<frame>parent</frame>
-    	<measure_direction>parent_to_child</measure_direction>
+    	<frame>sensor</frame>
     </force_torque>
   </plugin>
@@ -385,4 +378,10 @@
       </inertial>
     </link>
+    <xacro:if value="${gazebo}">
+      <gazebo reference="${side}_gripper_l_finger_tip">
+        <mu1>10000</mu1>
+        <mu2>10000</mu2>
+      </gazebo>
+    </xacro:if>
     <!-- Right finger joint -->
     <joint name="${side}_gripper_r_finger_joint" type="prismatic">
@@ -512,4 +511,10 @@
       </inertial>
     </link>
+    <xacro:if value="${gazebo}">
+      <gazebo reference="${side}_gripper_r_finger_tip">
+        <mu1>10000</mu1>
+        <mu2>10000</mu2>
+      </gazebo>
+    </xacro:if>
 <!-- Reference Joints, and links, non-visual, for transform references, and motion planning purposes -->
     <!--To connect this file with the sawyer_base.urdf.xacro a joint must be created between link "right_hand" in the latter file and "pneumatic_gripper_base", this way there is a transform between the robot last link and the End Of Arm Tooling in this file -->
@@ -530,18 +535,4 @@
     <!-- Pneumatic Gripper Tip link -->
     <link name="${side}_gripper_tip">
-      <inertial>
-        <origin xyz="0 0 0" rpy="0 0 0"/>
-        <mass value="2e-06"/>
-        <inertia ixx="1.1e-09" ixy="0" ixz="0" iyy="1.1e-09" iyz="0" izz="1.1e-09"/>
-      </inertial>
-    </link>
-    <!-- F/T sensor measure point at Tip link -->
-    <link name="${side}_ft_measure_tip">
-       <visual>
-              <origin rpy="0 0 0" xyz="0 0 0"/>
-        <geometry>
-          <box size="0.00001 0.00001 0.00001"/>
-        </geometry>
-      </visual>
       <inertial>
         <origin xyz="0 0 0" rpy="0 0 0"/>

Commit message: friction in gripper tips increased

File: intera_tools_description/urdf/smart_pneumatic_gripper/rethink_pneumatic_gripper.xacro (robot description, xacro)
@@ -380,6 +380,6 @@
     <xacro:if value="${gazebo}">
       <gazebo reference="${side}_gripper_l_finger_tip">
-        <mu1>10000</mu1>
-        <mu2>10000</mu2>
+        <mu1>100000.0</mu1>
+        <mu2>100000.0</mu2>
       </gazebo>
     </xacro:if>
@@ -513,6 +513,6 @@
     <xacro:if value="${gazebo}">
       <gazebo reference="${side}_gripper_r_finger_tip">
-        <mu1>10000</mu1>
-        <mu2>10000</mu2>
+        <mu1>100000.0</mu1>
+        <mu2>100000.0</mu2>
       </gazebo>
     </xacro:if>
@@ -540,4 +540,10 @@
         <inertia ixx="1.1e-09" ixy="0" ixz="0" iyy="1.1e-09" iyz="0" izz="1.1e-09"/>
       </inertial>
+      <visual>
+	<origin rpy="0 0 0" xyz="0 0 0"/>
+        <geometry>
+          <box size="0.0001 0.0001 0.0001"/>
+        </geometry>
+	</visual>
     </link>
     <!-- Gazebo References -->
