Commit message: pneumatic gripper inertias, CoM and masses updated for links

File: intera_tools_description/urdf/smart_pneumatic_gripper/rethink_pneumatic_gripper.xacro (robot description, xacro)
@@ -28,6 +28,6 @@
       <inertial>
         <!-- Sum Gripper Mass - for whole end effector, measured from end of plastic cuff -->
-        <mass value="1.902"/>
-        <origin rpy="0 0 0" xyz="0.0028 -0.0004 0.0343"/>
+        <mass value="2e-6"/>
+        <origin rpy="0 0 0" xyz="0.0 0.0 0.065"/>
         <inertia ixx="1e-08" ixy="0" ixz="0" iyy="1e-08" iyz="0" izz="1e-08"/>
       </inertial>
@@ -42,8 +42,7 @@
      <link name="${side}_connector_plate_base">
       <inertial>
-	      <origin xyz="0 0 0" rpy="${pi} 0 0" />
-        <mass value="0.387" />
-        <inertia ixx="0.0000292897"  ixy="6.1026E-08"  ixz="-1.5353186E-7"
-               iyy="0.0000296079"  iyz="-3.597884E-8" izz="0.0000508198" />
+	      <origin xyz="0 0 0.0151" rpy="${pi} 0 0" />
+        <mass value="0.35993" />
+        <inertia ixx="0.0002028057"  ixy="8.957633E-8"  ixz="-4.3426134E-7" iyy="0.0002052363"  iyz="1.243621E-8" izz="0.0003914837" />
       </inertial>
       <visual>
@@ -103,7 +102,7 @@
       </collision>
       <inertial>
-	      <origin rpy="${pi} 0 ${pi/2}" xyz="0 0 0"/>
-        <mass value="0.919"/>
-        <inertia ixx="0.0001756735" ixy="6.8322E-8" ixz="-2.7814E-8" iyy="0.0001757811" iyz="-9.2588E-8" izz="0.0002122946"/>
+	      <origin rpy="${pi} 0 ${pi/2}" xyz="0 0 ${ft_sensor_length*0.5}"/>
+        <mass value="0.91464"/>
+        <inertia ixx="0.0005579296" ixy="2.3164887E-7" ixz="3.046139E-8" iyy="0.000558405" iyz="-2.7494062E-7" izz="0.0009490083"/>
       </inertial>
     </link>
@@ -153,7 +152,7 @@
       </collision>
       <inertial>
-        <origin rpy="${-pi/2} 0 0" xyz="0.0 0.0 0.0"/>
-        <mass value="0.061"/>
-        <inertia ixx="0.0000418848" ixy="0" ixz="0" iyy="0.0000761051" iyz="0" izz="0.0000418848"/>
+        <origin rpy="${-pi/2} 0 0" xyz="0.0 0.0 ${adapter_top_length*0.5}"/>
+        <mass value="0.067"/>
+        <inertia ixx="0.0000352002" ixy="0" ixz="0" iyy="0.0000686304" iyz="0" izz="0.0000351976"/>
       </inertial>
     </link>
@@ -185,7 +184,7 @@
       </collision>
       <inertial>
-	<origin rpy="${-pi/2} 0 ${pi/2}" xyz="0.0 0.0 0.0"/>
-        <mass value="0.098"/>
-        <inertia ixx="0.0000721906" ixy="0" ixz="0" iyy="0.0001202265" iyz="0" izz="0.0000723151"/>
+	<origin rpy="${-pi/2} 0 ${pi/2}" xyz="0.0 0.0 ${adapter_bottom_length*0.5}"/>
+        <mass value="0.102"/>
+        <inertia ixx="0.0000569055" ixy="0" ixz="0" iyy="0.0001084165" iyz="0" izz="0.0000570176"/>
       </inertial>
     </link>
@@ -225,7 +224,7 @@
       </collision>
       <inertial>
-	      <origin rpy="${pi/2} 0 0" xyz="0.0 0.0 0.0"/>
-        <mass value="0.311"/>
-        <inertia ixx="0.0000330475" ixy="1.31E-8" ixz="0" iyy="0.0000176978" iyz="0" izz="0.0000203961"/>
+	      <origin rpy="${pi/2} 0 0" xyz="0.0 0.0 0.017"/>
+        <mass value="0.359"/>
+        <inertia ixx="0.0001531281" ixy="-2.4547146E-7" ixz="-3.4522E-10" iyy="0.0001380478" iyz="-2.6043E-10" izz="0.0000544404"/>
       </inertial>
     </link>
@@ -276,7 +275,7 @@
       </collision>
       <inertial>
-	<origin rpy="${pi/2} 0 0" xyz="0 0.0295 0"/>
-        <mass value="0.010"/>
-        <inertia ixx="0.0000013187" ixy="0" ixz="0" iyy="0.0000012511" iyz="2.8731E-7" izz="2.2756E-7"/>
+	      <origin rpy="${pi/2} 0 0" xyz="0 0.0435 0.005"/>
+        <mass value="0.011"/>
+        <inertia ixx="9.2817609E-7" ixy="0" ixz="0" iyy="0.0000010234" iyz="-3.31923299E-8" izz="3.3665975E-7"/>
       </inertial>
     </link>
@@ -315,7 +314,7 @@
       </collision>
       <inertial>
-	      <origin rpy="0 0 ${pi/2}" xyz="0 0.0185 0"/>
-        <mass value="0.029"/>
-        <inertia ixx="0.00000151" ixy="-1.23E-12" ixz="0.0000025354" iyy="0.000042463" iyz="-1.23E-12" izz="0.0000433196"/>
+	      <origin rpy="0 0 ${pi/2}" xyz="0 0.0495 0.003"/>
+        <mass value="0.027"/>
+        <inertia ixx="0.0000012665" ixy="-1.23E-12" ixz="1.166012E-8" iyy="0.0000160553" iyz="-1.23E-12" izz="0.0000171552"/>
       </inertial>
     </link>
@@ -344,7 +343,7 @@
       </collision>
       <inertial>
-	<origin rpy="0 0 ${pi/2}" xyz="0 -0.0035 0"/>
-        <mass value="0.037"/>
-        <inertia ixx="0.0000683111" ixy="-1.24623E-9" ixz="0.0000038251" iyy="0.0000668321" iyz="-1.738481E-8" izz="0.0000031831"/>
+	      <origin rpy="0 0 ${pi/2}" xyz="0.0 0.00 0.035"/>
+        <mass value="0.036"/>
+        <inertia ixx="0.0000239168" ixy="3.1961E-10" ixz="-9.4649889E-7" iyy="0.0000219249" iyz="-2.81633999E-9" izz="00.0000026702"/>
       </inertial>
     </link>
@@ -373,7 +372,7 @@
       </collision>
       <inertial>
-	      <origin rpy="0 0 ${pi/2}" xyz="0 -0.0035 ${0.0726-((tip_slot_pos-1)*0.015)}"/>
-        <mass value="0.040"/>
-        <inertia ixx="0.0000064492" ixy="-2.802891E-8" ixz="-2.65457E-9" iyy="0.0000019488" iyz="1.4972E-10" izz="0.0000057675"/>
+	      <origin rpy="0 0 ${pi/2}" xyz="0 -0.0085 ${0.0726-((tip_slot_pos-1)*0.015)}"/>
+        <mass value="0.0138"/>
+        <inertia ixx="0.0000049904" ixy="0" ixz="0" iyy="0.0000011238" iyz="0" izz="0.0000040782"/>
       </inertial>
     </link>
@@ -409,7 +408,7 @@
       </collision>
       <inertial>
-	      <origin rpy="${pi/2} 0 ${pi}" xyz="0 -0.0295 0"/>
-        <mass value="0.010"/>
-        <inertia ixx="0.0000013187" ixy="0" ixz="0" iyy="0.0000012511" iyz="2.8731E-7" izz="2.2756E-7"/>
+	      <origin rpy="${pi/2} 0 ${pi}" xyz="0 -0.0435 0.005"/>
+        <mass value="0.011"/>
+        <inertia ixx="9.2817609E-7" ixy="0" ixz="0" iyy="0.0000010234" iyz="-3.31923299E-8" izz="3.3665975E-7"/>
       </inertial>
     </link>
@@ -448,7 +447,7 @@
       </collision>
       <inertial>
-	      <origin rpy="0 0 ${-pi/2}" xyz="0 -0.0185 0"/>
-        <mass value="0.029"/>
-        <inertia ixx="0.00000151" ixy="-1.23E-12" ixz="0.0000025354" iyy="0.000042463" iyz="-1.23E-12" izz="0.0000433196"/>
+	      <origin rpy="0 0 ${-pi/2}" xyz="0 -0.0495 0.003"/>
+        <mass value="0.027"/>
+        <inertia ixx="0.0000012665" ixy="-1.23E-12" ixz="1.166012E-8" iyy="0.0000160553" iyz="-1.23E-12" izz="0.0000171552"/>
       </inertial>
     </link>
@@ -477,7 +476,7 @@
       </collision>
       <inertial>
-	      <origin rpy="0 0 ${-pi/2}" xyz="0 0.0035 0"/>
-        <mass value="0.037"/>
-        <inertia ixx="0.0000683111" ixy="-1.24623E-9" ixz="0.0000038251" iyy="0.0000668321" iyz="-1.738481E-8" izz="0.0000031831"/>
+	      <origin rpy="0 0 ${-pi/2}" xyz="0 0.0 0.035"/>
+        <mass value="0.036"/>
+        <inertia ixx="0.0000239168" ixy="3.1961E-10" ixz="-9.4649889E-7" iyy="0.0000219249" iyz="-2.81633999E-9" izz="00.0000026702"/>
       </inertial>
     </link>
@@ -506,7 +505,7 @@
       </collision>
       <inertial>
-	      <origin rpy="0 0 ${-pi/2}" xyz="0 0.0035 ${0.0726-((tip_slot_pos-1)*0.015)}"/>
-        <mass value="0.040"/>
-        <inertia ixx="0.0000064492" ixy="-2.802891E-8" ixz="-2.65457E-9" iyy="0.0000019488" iyz="1.4972E-10" izz="0.0000057675"/>
+	      <origin rpy="0 0 ${-pi/2}" xyz="0 0.0085 ${0.0726-((tip_slot_pos-1)*0.015)}"/>
+        <mass value="0.0138"/>
+        <inertia ixx="0.0000049904" ixy="0" ixz="0" iyy="0.0000011238" iyz="0" izz="0.0000040782"/>
       </inertial>
     </link>

Commit message: limits updated for virtual ft sensor

File: intera_tools_description/urdf/smart_pneumatic_gripper/rethink_pneumatic_gripper.xacro (robot description, xacro)
@@ -116,5 +116,5 @@
          <child  link="${side}_adapter_top" />
          <axis xyz="1 0 0"/>
-         <limit lower="-0.001" upper="0.001" effort="1000" velocity="1000"/>
+         <limit lower="-0.01" upper="0.01" effort="100" velocity="10"/>
     </joint>
     <gazebo reference="${side}_ft_sensor_adapter_top_joint">
